File: hardware/pcb/miniCO2/miniCO2.kicad_pcb (KiCad board)
At the start: 4 copper layers, 17 x 18.5 mm, 12 parts, among them J1 USB_A, J2 Conn_01x04_Socket, SW1 SW_Push, U1 ATSAMD21E18A-M, U2 AP2112K-3.3, U3 SCD40-D-R2

Commit message: Fix D1, D2 footprints
Parts:
- U1: value ATSAMD21E18A-M -> ATSAMD21E17A-MUT
- moved D1 7.62 mm to (137.6, 95.1)
- moved D2 7.58 mm to (145.2, 95.1)
Connections:
- D1 pad 1: Net-(D1-DOUT) -> DIN
- D1 pad 2: GND -> +3.3V
- D1 pad 3: DIN -> Net-(D1-DOUT)
- D1 pad 4: +3.3V -> GND
- D2 pad 1: unconnected-(D2-DOUT-Pad1) -> Net-(D1-DOUT)
- D2 pad 2: GND -> +3.3V
- D2 pad 3: Net-(D1-DOUT) -> unconnected-(D2-DOUT-Pad3)
- D2 pad 4: +3.3V -> GND
Routing:
- net DIN: track 11.5 -> 7.94 mm
- net Net-(D1-DOUT): track 7.28 -> 8.21 mm, vias 2 -> 0
Changed lines of the file:
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@@
 	(net 3 "DIN")
 	(net 4 "+3.3V")
-	(net 5 "unconnected-(D2-DOUT-Pad1)")
+	(net 5 "unconnected-(D2-DOUT-Pad3)")
 	(net 6 "unconnected-(U1-PA00-Pad1)")
 	(net 7 "unconnected-(U1-PA01-Pad2)")
@@
 			)
 		)
-		(property "LCSC Part #" "C2763086"
+		(property "LCSC Part #" " C2763083"
 			(at 0 0 0)
 			(unlocked yes)
@@
 	(footprint "MiniCO2:WS2812C-4020"
 		(layer "F.Cu")
-		(at 137.6414 95.031262 180)
+		(at 145.2219 95.081262 180)
 		(property "Reference" "D2"
 			(at 3.424 -0.254 0)
@@
 			)
 		)
-		(property "LCSC Part #" "C5149201"
+		(property "LCSC Part #" "C4154870"
 			(at 0 0 180)
 			(unlocked yes)
@@
 			)
 		)
-		(property ki_fp_filters "LED*SK6805*PLCC*2.4x2.7mm*P1.3mm*")
 		(sheetname "Root")
 		(sheetfile "miniCO2.kicad_sch")
@@
 		)
 		(fp_text user "${REFERENCE}"
-			(at -0.0805 -0.2 0)
+			(at 0.075 -0.55 0)
 			(unlocked yes)
 			(layer "F.Fab")
@@
 			(size 0.42 1.3)
 			(layers "F.Cu" "F.Paste" "F.Mask")
-			(net 5 "unconnected-(D2-DOUT-Pad1)")
-			(pinfunction "DOUT")
-			(pintype "output")
+			(net 1 "Net-(D1-DOUT)")
+			(pinfunction "DIN")
+			(pintype "input")
 			(thermal_bridge_angle 45)
 		)
@@
 			(size 0.42 1.3)
 			(layers "F.Cu" "F.Paste" "F.Mask")
-			(net 2 "GND")
-			(pinfunction "VSS")
+			(net 4 "+3.3V")
+			(pinfunction "VDD")
 			(pintype "power_in")
 			(thermal_bridge_angle 45)
@@
 			(size 0.42 1.3)
 			(layers "F.Cu" "F.Paste" "F.Mask")
-			(net 1 "Net-(D1-DOUT)")
-			(pinfunction "DIN")
-			(pintype "input")
+			(net 5 "unconnected-(D2-DOUT-Pad3)")
+			(pinfunction "DOUT")
+			(pintype "output")
 			(thermal_bridge_angle 45)
 		)
@@
 			(size 0.42 1.3)
 			(layers "F.Cu" "F.Paste" "F.Mask")
-			(net 4 "+3.3V")
-			(pinfunction "VDD")
+			(net 2 "GND")
+			(pinfunction "VSS")
 			(pintype "power_in")
 			(thermal_bridge_angle 45)
@@
 	(footprint "MiniCO2:WS2812C-4020"
 		(layer "F.Cu")
-		(at 145.2414 95.031262 180)
+		(at 137.6219 95.081262 180)
 		(property "Reference" "D1"
 			(at -3.048 0.508 180)
@@
 			)
 		)
-		(property "LCSC Part #" "C5149201"
+		(property "LCSC Part #" "C4154870"
 			(at 0 0 180)
 			(unlocked yes)
@@
 			)
 		)
-		(property ki_fp_filters "LED*SK6805*PLCC*2.4x2.7mm*P1.3mm*")
 		(sheetname "Root")
 		(sheetfile "miniCO2.kicad_sch")
@@
 		)
 		(fp_text user "${REFERENCE}"
-			(at -0.0805 -0.1 0)
+			(at 4.25 -2.6 0)
 			(unlocked yes)
 			(layer "F.Fab")
@@
 			(size 0.42 1.3)
 			(layers "F.Cu" "F.Paste" "F.Mask")
-			(net 1 "Net-(D1-DOUT)")
-			(pinfunction "DOUT")
-			(pintype "output")
+			(net 3 "DIN")
+			(pinfunction "DIN")
+			(pintype "input")
 			(thermal_bridge_angle 45)
 		)
@@
 			(size 0.42 1.3)
 			(layers "F.Cu" "F.Paste" "F.Mask")
-			(net 2 "GND")
-			(pinfunction "VSS")
+			(net 4 "+3.3V")
+			(pinfunction "VDD")
 			(pintype "power_in")
 			(thermal_bridge_angle 45)
@@
 			(size 0.42 1.3)
 			(layers "F.Cu" "F.Paste" "F.Mask")
-			(net 3 "DIN")
-			(pinfunction "DIN")
-			(pintype "input")
+			(net 1 "Net-(D1-DOUT)")
+			(pinfunction "DOUT")
+			(pintype "output")
 			(thermal_bridge_angle 45)
 		)
@@
 			(size 0.42 1.3)
 			(layers "F.Cu" "F.Paste" "F.Mask")
-			(net 4 "+3.3V")
-			(pinfunction "VDD")
+			(net 2 "GND")
+			(pinfunction "VSS")
 			(pintype "power_in")
 			(thermal_bridge_angle 45)
@@
 			)
 		)
-		(property "Value" "ATSAMD21E18A-M"
+		(property "Value" "ATSAMD21E17A-MUT"
 			(at -10.35 0.3088 0)
 			(layer "F.Fab")
@@
 			)
 		)
-		(property "LCSC Part #" "C2052801"
+		(property "LCSC Part #" "3A991A2"
 			(at 0 0 180)
 			(unlocked yes)
@@
 	)
 	(segment
-		(start 143.9664 95.031262)
-		(end 143.3958 95.031262)
-		(width 0.15)
-		(layer "F.Cu")
-		(net 1)
-	)
-	(segment
-		(start 143.3958 95.031262)
-		(end 143.3718 95.055262)
+		(start 138.3969 96.206262)
+		(end 143.6469 96.206262)
 		(width 0.15)
 		(layer "F.Cu")
@@
 	)
 	(segment
-		(start 139.157 93.937662)
-		(end 138.62 93.937662)
+		(start 143.6469 96.206262)
+		(end 143.9469 95.906262)
 		(width 0.15)
 		(layer "F.Cu")
@@
 	)
 	(segment
-		(start 138.62 93.937662)
-		(end 137.9664 94.591262)
+		(start 138.0469 95.081262)
+		(end 138.0469 95.856262)
 		(width 0.15)
 		(layer "F.Cu")
 		(net 1)
 	)
-	(via
-		(at 139.157 93.937662)
-		(size 0.4)
-		(drill 0.3)
-		(layers "F.Cu" "B.Cu")
-		(net 1)
-	)
-	(via
-		(at 143.3718 95.055262)
-		(size 0.4)
-		(drill 0.3)
-		(layers "F.Cu" "B.Cu")
-		(net 1)
-	)
-	(segment
-		(start 139.157 93.937662)
-		(end 142.2542 93.937662)
-		(width 0.15)
-		(layer "In2.Cu")
-		(net 1)
-	)
 	(segment
-		(start 142.2542 93.937662)
-		(end 143.3718 95.055262)
+		(start 143.9469 95.906262)
+		(end 143.9469 95.081262)
 		(width 0.15)
-		(layer "In2.Cu")
+		(layer "F.Cu")
 		(net 1)
 	)
 	(segment
-		(start 143.3718 95.055262)
-		(end 143.2718 95.055262)
+		(start 138.0469 95.856262)
+		(end 138.3969 96.206262)
 		(width 0.15)
-		(layer "In2.Cu")
+		(layer "F.Cu")
 		(net 1)
 	)
@@
 	)
 	(segment
-		(start 139.197564 91.872462)
-		(end 138.5219 91.872462)
-		(width 0.2)
-		(layer "F.Cu")
-		(net 3)
-	)
-	(segment
-		(start 139.676482 92.35138)
-		(end 139.197564 91.872462)
-		(width 0.2)
+		(start 139.1881 91.872462)
+		(end 139.6969 92.381262)
+		(width 0.15)
 		(layer "F.Cu")
 		(net 3)
 	)
 	(segment
-		(start 145.6664 95.756262)
-		(end 145.6664 95.031262)
-		(width 0.2)
+		(start 136.3469 96.031262)
+		(end 136.3469 95.081262)
+		(width 0.15)
 		(layer "F.Cu")
 		(net 3)
 	)
 	(segment
-		(start 146.0414 96.131262)
-		(end 145.6664 95.756262)
-		(width 0.2)
+		(start 138.5219 91.872462)
+		(end 139.1881 91.872462)
+		(width 0.15)
 		(layer "F.Cu")
 		(net 3)
 	)
 	(via
-		(at 146.0414 96.131262)
+		(at 136.3469 96.031262)
 		(size 0.4)
 		(drill 0.3)
@@
 	)
 	(via
-		(at 139.676482 92.35138)
+		(at 139.6969 92.381262)
 		(size 0.4)
 		(drill 0.3)
@@
 	)
 	(segment
-		(start 139.676482 92.35138)
-		(end 143.971518 92.35138)
-		(width 0.2)
+		(start 136.3469 96.031262)
+		(end 136.3469 95.967721)
+		(width 0.15)
 		(layer "In1.Cu")
 		(net 3)
 	)
 	(segment
-		(start 146.0414 94.421262)
-		(end 146.0414 96.131262)
-		(width 0.2)
+		(start 136.3469 95.967721)
+		(end 137.233359 95.081262)
+		(width 0.15)
 		(layer "In1.Cu")
 		(net 3)
 	)
 	(segment
-		(start 143.971518 92.35138)
-		(end 146.0414 94.421262)
-		(width 0.2)
+		(start 138.0719 95.081262)
+		(end 139.7844 93.368762)
+		(width 0.15)
+		(layer "In1.Cu")
+		(net 3)
+	)
+	(segment
+		(start 137.233359 95.081262)
+		(end 138.0719 95.081262)
+		(width 0.15)
+		(layer "In1.Cu")
+		(net 3)
+	)
+	(segment
+		(start 139.7844 92.468762)
+		(end 139.6969 92.381262)
+		(width 0.15)
+		(layer "In1.Cu")
+		(net 3)
+	)
+	(segment
+		(start 139.7844 93.368762)
+		(end 139.7844 92.468762)
+		(width 0.15)
 		(layer "In1.Cu")
 		(net 3)
@@
 	)
 	(segment
-		(start 138.9164 95.031262)
-		(end 139.6174 95.031262)
-		(width 0.8)
+		(start 137.1969 95.081262)
+		(end 137.1969 95.931262)
+		(width 0.5)
 		(layer "F.Cu")
 		(net 4)
@@
 	)
 	(segment
-		(start 147.8969 82.973062)
-		(end 148.7819 83.858062)
-		(width 0.8)
+		(start 144.7969 95.081262)
+		(end 144.7969 96.006262)
+		(width 0.5)
 		(layer "F.Cu")
 		(net 4)
 	)
 	(segment
-		(start 148.6914 90.238862)
-		(end 147.943662 90.238862)
+		(start 147.8969 82.973062)
+		(end 148.7819 83.858062)
 		(width 0.8)
 		(layer "F.Cu")
@@
 	)
 	(segment
-		(start 139.6174 95.031262)
-		(end 139.6414 95.007262)
+		(start 148.6914 90.238862)
+		(end 147.943662 90.238862)
 		(width 0.8)
 		(layer "F.Cu")
@@
 	)
 	(segment
-		(start 147.2219 95.431262)
-		(end 146.8219 95.031262)
+		(start 144.7969 96.006262)
+		(end 144.8219 96.031262)
 		(width 0.5)
 		(layer "F.Cu")
@@
 	)
 	(segment
+		(start 137.1969 95.931262)
+		(end 137.1969 95.919122)
+		(width 0.5)
+		(layer "F.Cu")
+		(net 4)
+	)
+	(segment
 		(start 147.943662 90.238862)
 		(end 147.4684 89.7636)
@@
 		(net 4)
 	)
-	(segment
-		(start 139.6174 95.055262)
-		(end 139.6414 95.031262)
-		(width 0.8)
-		(layer "F.Cu")
-		(net 4)
-	)
-	(segment
-		(start 146.8219 95.031262)
-		(end 146.5164 95.031262)
-		(width 0.5)
-		(layer "F.Cu")
+	(via
+		(at 144.8219 96.031262)
+		(size 0.4)
+		(drill 0.3)
+		(layers "F.Cu" "B.Cu")
 		(net 4)
 	)
@@
 	)
 	(via
-		(at 147.2219 95.431262)
-		(size 0.8)
-		(drill 0.4)
-		(layers "F.Cu" "B.Cu")
-		(net 4)
-	)
-	(via
-		(at 139.6414 95.007262)
-		(size 0.8)
-		(drill 0.4)
+		(at 137.1969 95.931262)
+		(size 0.4)
+		(drill 0.3)
 		(layers "F.Cu" "B.Cu")
 		(net 4)
