File: hardware/pcb/miniCO2/ESP32/display.kicad_sch (KiCad schematic)
At the start: 18 parts, among them J2 Conn_01x18, Q2 Si1308EDL

Commit message: Modifications before sending to production
Parts:
- C11, C12, C13, C5, C7: value 2.2uF -> 2.2uF/10V; LCSC Part # C386031 -> C335106
- C14: value 100n -> 100n/25V; LCSC C1525 -> (none); LCSC Part # C76934 -> C181047
- C15, C18: value 4.7uF/25V -> 4.7uF/35V; LCSC Part # C69335 -> C162274
- C17, C6: value 1uF/25V -> 1uF/50V; LCSC Part # C5673 -> C342951
- J2: value Conn_01x18 -> FPC 18POS 0.5mm; LCSC Part # (none) -> C397324
- R4: LCSC Part # C295786 -> C473450
- R5: LCSC Part # C473517 -> C270323
Other:
- note removed: "1uF under bias"
Changed lines of the file:
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@@
-		)
-	)
-	(text "1uF under bias"
-		(exclude_from_sim no)
-		(at 138.938 60.198 0)
-		(effects
-			(font
-				(size 1.27 1.27)
-			)
 		)
 	)
@@
 			)
 		)
-		(property "LCSC Part #" "C295786"
+		(property "LCSC Part #" "C473450"
 			(at 140.97 96.52 0)
 			(effects
@@
 			)
 		)
-		(property "Value" "2.2uF"
+		(property "Value" "2.2uF/10V"
 			(at 118.11 123.19 0)
 			(effects
@@
 			)
 		)
-		(property "LCSC Part #" "C386031"
+		(property "LCSC Part #" "C335106"
 			(at 114.3 121.92 0)
 			(effects
@@
 			)
 		)
-		(property "LCSC Part #" "C473517"
+		(property "LCSC Part #" "C270323"
 			(at 148.59 96.52 0)
 			(effects
@@
 			)
 		)
-		(property "Value" "2.2uF"
+		(property "Value" "2.2uF/10V"
 			(at 106.68 123.19 0)
 			(effects
@@
 			)
 		)
-		(property "LCSC Part #" "C386031"
+		(property "LCSC Part #" "C335106"
 			(at 102.87 121.92 0)
 			(effects
@@
 			)
 		)
-		(property "Value" "Conn_01x18"
+		(property "Value" "FPC 18POS 0.5mm"
 			(at 97.79 97.79 0)
 			(effects
@@
 		)
 		(property "Description" "Generic connector, single row, 01x18, script generated (kicad-library-utils/schlib/autogen/connector/)"
+			(at 97.79 71.12 0)
+			(effects
+				(font
+					(size 1.27 1.27)
+				)
+				(hide yes)
+			)
+		)
+		(property "LCSC Part #" "C397324"
 			(at 97.79 71.12 0)
 			(effects
@@
 			)
 		)
-		(property "Value" "2.2uF"
+		(property "Value" "2.2uF/10V"
 			(at 80.01 123.19 0)
 			(effects
@@
 			)
 		)
-		(property "LCSC Part #" "C386031"
+		(property "LCSC Part #" "C335106"
 			(at 76.2 121.92 0)
 			(effects
@@
 			)
 		)
-		(property "Value" "100n"
+		(property "Value" "100n/25V"
 			(at 130.81 124.46 0)
 			(effects
@@
 			)
 		)
-		(property "LCSC" "C1525"
+		(property "LCSC" ""
 			(at 130.81 121.92 0)
 			(effects
@@
 			)
 		)
-		(property "LCSC Part #" "C76934"
+		(property "LCSC Part #" "C181047"
 			(at 130.81 121.92 0)
 			(effects
@@
 			)
 		)
-		(property "Value" "2.2uF"
+		(property "Value" "2.2uF/10V"
 			(at 93.98 123.19 0)
 			(effects
@@
 			)
 		)
-		(property "LCSC Part #" "C386031"
+		(property "LCSC Part #" "C335106"
 			(at 90.17 121.92 0)
 			(effects
@@
 		)
 		(property "Value" "Si1308EDL"
-			(at 204.978 90.424 0)
+			(at 149.352 83.058 0)
 			(effects
 				(font
@@
 		)
 		(property "Value" "NSR05F30NXT5G"
-			(at 204.216 71.374 0)
+			(at 158.75 71.628 0)
 			(effects
 				(font
@@
 			)
 		)
-		(property "Value" "4.7uF/25V"
+		(property "Value" "4.7uF/35V"
 			(at 135.382 66.04 0)
 			(effects
@@
 			)
 		)
-		(property "LCSC Part #" "C69335"
+		(property "LCSC Part #" "C162274"
 			(at 148.59 64.77 0)
 			(effects
@@
 		)
 		(property "Value" "NSR05F30NXT5G"
-			(at 207.01 63.246 0)
+			(at 160.02 60.198 0)
 			(effects
 				(font
@@
 			)
 		)
-		(property "Value" "1uF/25V"
+		(property "Value" "1uF/50V"
 			(at 170.18 81.28 0)
 			(effects
@@
 			)
 		)
-		(property "LCSC Part #" "C5673"
+		(property "LCSC Part #" "C342951"
 			(at 166.37 80.01 0)
 			(effects
@@
 		)
 		(property "Value" "NSR05F30NXT5G"
-			(at 205.74 56.642 0)
+			(at 160.02 52.578 0)
 			(effects
 				(font
@@
 			)
 		)
-		(property "Value" "1uF/25V"
+		(property "Value" "1uF/50V"
 			(at 173.99 62.23 0)
 			(effects
@@
 			)
 		)
-		(property "LCSC Part #" "C5673"
+		(property "LCSC Part #" "C342951"
 			(at 170.18 60.96 0)
 			(effects
@@
 			)
 		)
-		(property "Value" "2.2uF"
+		(property "Value" "2.2uF/10V"
 			(at 67.31 123.19 0)
 			(effects
@@
 			)
 		)
-		(property "LCSC Part #" "C386031"
+		(property "LCSC Part #" "C335106"
 			(at 63.5 121.92 0)
 			(effects
@@
 			)
 		)
-		(property "Value" "4.7uF/25V"
+		(property "Value" "4.7uF/35V"
 			(at 115.062 81.28 0)
 			(effects
@@
 			)
 		)
-		(property "LCSC Part #" "C69335"
+		(property "LCSC Part #" "C162274"
 			(at 128.27 80.01 0)
 			(effects
