File: hardware/pcb/miniCO2/ESP32/untitled.kicad_sch (KiCad schematic)
At the start: 26 parts, among them J1 USB_C_16P, SW3 MK-12C03-G015, U5 SLM6401, U6 LM66100DCK, U7 LM66100DCK, U8 TPS62172DSG

Commit message: Modifications before sending to production
Parts:
- removed D5: CUS10S30,H3F, Diode_SMD:D_SOD-323, symbol Device:D_Schottky
- C1, C19, C2, C3: value 22uF -> 22uF/25V; LCSC Part # C86816 -> C6119899
- C10: value 100n -> 100n/25V; LCSC C1525 -> (none); LCSC Part # C76934 -> C181047
- C9: value 10n -> 10n/50V; LCSC Part # C282517 -> C57112
- D4: value ESD9B5.0ST5G -> ESD9L5.0ST5G-ES; LCSC Part # C3008065 -> C5199180
- D8: LCSC Part # C965791 -> C510300
- FB1: value BLM15PX471SN1D -> TDK MPZ1005S121CT000; LCSC Part # C333978 -> C107331
- H1, H2: now not fitted
- R1, R2, R3: LCSC Part # C274341 -> C270344
- R8: LCSC Part # C163457 -> C25908
Connections:
- net VBUS: now also C10.1, FB1.2
Changed lines of the file:
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@@
 	(wire
 		(pts
-			(xy 151.13 31.75) (xy 157.48 31.75)
-		)
-		(stroke
-			(width 0)
-			(type default)
-		)
-	)
-	(wire
-		(pts
 			(xy 157.48 31.75) (xy 157.48 33.02)
 		)
@@
 	(wire
 		(pts
-			(xy 139.7 31.75) (xy 143.51 31.75)
+			(xy 139.7 31.75) (xy 157.48 31.75)
 		)
 		(stroke
@@
 			)
 		)
-		(property "Value" "10n"
+		(property "Value" "10n/50V"
 			(at 132.08 36.322 0)
 			(effects
@@
 			)
 		)
-		(property "LCSC Part #" "C282517"
+		(property "LCSC Part #" "C57112"
 			(at 129.54 35.56 0)
 			(effects
@@
 			)
 		)
-		(property "Value" "ESD9B5.0ST5G"
-			(at 103.378 58.928 90)
+		(property "Value" "ESD9L5.0ST5G-ES"
+			(at 107.696 38.608 90)
 			(effects
 				(font
@@
 			)
 		)
-		(property "Datasheet" "https://www.onsemi.com/pub/Collateral/ESD9B-D.PDF"
+		(property "Datasheet" "https://www.lcsc.com/datasheet/lcsc_datasheet_2412061751_ElecSuper-ESD9L5-0ST5G-ES_C5199180.pdf"
 			(at 123.19 35.56 0)
 			(effects
@@
 			)
 		)
-		(property "Description" "ESD protection diode, 5.0Vrwm, SOD-923"
+		(property "Description" "ESD protection diode, 6.0V, SOD-923"
 			(at 123.19 35.56 0)
 			(effects
@@
 			)
 		)
-		(property "LCSC Part #" "C3008065"
+		(property "LCSC Part #" "C5199180"
 			(at 123.19 35.56 0)
 			(effects
@@
 		)
 		(property "Value" "6V 750mA 40A 1.5A"
-			(at 126.746 18.034 90)
+			(at 117.094 28.194 90)
 			(effects
 				(font
@@
 			)
 		)
-		(property "Value" "22uF"
+		(property "Value" "22uF/25V"
 			(at 88.646 116.586 0)
 			(effects
@@
 			)
 		)
-		(property "LCSC Part #" "C86816"
+		(property "LCSC Part #" "C6119899"
 			(at 81.28 115.57 0)
 			(effects
@@
 			)
 		)
-		(property "LCSC Part #" "C274341"
+		(property "LCSC Part #" "C270344"
 			(at 40.64 105.41 0)
 			(effects
@@
 			)
 		)
-		(property "LCSC Part #" "C163457"
+		(property "LCSC Part #" "C25908"
 			(at 74.93 123.19 0)
 			(effects
@@
 		(in_bom no)
 		(on_board yes)
-		(dnp no)
+		(dnp yes)
 		(fields_autoplaced yes)
 		(property "Reference" "H2"
@@
 			)
 		)
-		(property "Datasheet" "https://www.lcsc.com/datasheet/lcsc_datasheet_2410121310_XINGLIGHT-XL-1005UOC_C965791.pdf"
+		(property "Datasheet" "https://www.lcsc.com/datasheet/lcsc_datasheet_2111161030_ROHM-Semicon-SML-P11UTT86R_C510300.pdf"
 			(at 40.64 113.03 0)
 			(effects
@@
 			)
 		)
-		(property "LCSC Part #" "C965791"
+		(property "LCSC Part #" "C510300"
 			(at 40.64 113.03 90)
 			(effects
@@
 		(dnp no)
 		(property "Reference" "C3"
-			(at 153.162 35.56 0)
+			(at 163.068 35.56 0)
 			(effects
 				(font
@@
 			)
 		)
-		(property "Value" "22uF"
-			(at 153.924 37.846 0)
+		(property "Value" "22uF/25V"
+			(at 169.672 37.592 0)
 			(effects
 				(font
@@
 			)
 		)
-		(property "LCSC Part #" "C86816"
+		(property "LCSC Part #" "C6119899"
 			(at 157.48 36.83 0)
 			(effects
@@
 		(in_bom no)
 		(on_board yes)
-		(dnp no)
+		(dnp yes)
 		(fields_autoplaced yes)
 		(property "Reference" "H1"
@@
 			)
 		)
-		(property "Value" "100n"
+		(property "Value" "100n/25V"
 			(at 142.748 37.338 0)
 			(effects
@@
 			)
 		)
-		(property "LCSC" "C1525"
+		(property "LCSC" ""
 			(at 139.7 35.56 0)
 			(effects
@@
 			)
 		)
-		(property "LCSC Part #" "C76934"
+		(property "LCSC Part #" "C181047"
 			(at 139.7 35.56 0)
 			(effects
@@
 			)
 		)
-		(property "Value" "22uF"
+		(property "Value" "22uF/25V"
 			(at 184.404 105.156 0)
 			(effects
@@
 			)
 		)
-		(property "LCSC Part #" "C86816"
+		(property "LCSC Part #" "C6119899"
 			(at 187.96 104.14 0)
 			(effects
@@
 			)
 		)
-		(property "Value" "22uF"
+		(property "Value" "22uF/25V"
 			(at 235.712 105.664 0)
 			(effects
@@
 			)
 		)
-		(property "LCSC Part #" "C86816"
+		(property "LCSC Part #" "C6119899"
 			(at 227.33 104.14 0)
 			(effects
@@
 			)
 		)
-		(property "Value" "BLM15PX471SN1D"
-			(at 155.448 19.558 90)
+		(property "Value" "TDK MPZ1005S121CT000"
+			(at 136.144 26.67 90)
 			(effects
 				(font
@@
 			)
 		)
-		(property "Datasheet" "https://www.lcsc.com/datasheet/lcsc_datasheet_1912111437_Murata-Electronics-BLM15PX471SN1D_C333978.pdf"
+		(property "Datasheet" "https://www.lcsc.com/datasheet/lcsc_datasheet_2412191506_TDK-MPZ1005S121CT000_C107331.pdf"
 			(at 135.89 31.75 0)
 			(effects
@@
 			)
 		)
-		(property "LCSC" ""
-			(at 135.89 31.75 90)
-			(effects
-				(font
-					(size 1.27 1.27)
-				)
-				(hide yes)
-			)
-		)
-		(property "LCSC Part #" "C333978"
+		(property "LCSC Part #" "C107331"
 			(at 135.89 31.75 0)
 			(effects
@@
 			)
 		)
-		(property "LCSC Part #" "C274341"
+		(property "LCSC Part #" "C270344"
 			(at 80.01 44.45 0)
 			(effects
@@
 	)
 	(symbol
-		(lib_id "Device:D_Schottky")
-		(at 147.32 31.75 180)
-		(unit 1)
-		(exclude_from_sim no)
-		(in_bom yes)
-		(on_board yes)
-		(dnp no)
-		(property "Reference" "D5"
-			(at 147.32 28.575 0)
-			(effects
-				(font
-					(size 1.27 1.27)
-				)
-			)
-		)
-		(property "Value" "CUS10S30,H3F"
-			(at 173.736 16.51 0)
-			(effects
-				(font
-					(size 1.27 1.27)
-				)
-			)
-		)
-		(property "Footprint" "Diode_SMD:D_SOD-323"
-			(at 147.32 31.75 0)
-			(effects
-				(font
-					(size 1.27 1.27)
-				)
-				(hide yes)
-			)
-		)
-		(property "Datasheet" "https://www.lcsc.com/datasheet/lcsc_datasheet_2410121958_TOSHIBA-CUS10S30-H3F_C146335.pdf"
-			(at 147.32 31.75 0)
-			(effects
-				(font
-					(size 1.27 1.27)
-				)
-				(hide yes)
-			)
-		)
-		(property "Description" ""
-			(at 147.32 31.75 0)
-			(effects
-				(font
-					(size 1.27 1.27)
-				)
-				(hide yes)
-			)
-		)
-		(property "MPN " "CUS10S30,H3F"
-			(at 147.32 31.75 0)
-			(effects
-				(font
-					(size 1.27 1.27)
-				)
-				(hide yes)
-			)
-		)
-		(property "JLCPCB_CORRECTION" ""
-			(at 147.32 31.75 0)
-			(effects
-				(font
-					(size 1.27 1.27)
-				)
-				(hide yes)
-			)
-		)
-		(property "LCSC" ""
-			(at 147.32 31.75 0)
-			(effects
-				(font
-					(size 1.27 1.27)
-				)
-				(hide yes)
-			)
-		)
-		(property "LCSC Part #" "C146335"
-			(at 147.32 31.75 0)
-			(effects
-				(font
-					(size 1.27 1.27)
-				)
-				(hide yes)
-			)
-		)
-		(pin "1"
-		)
-		(pin "2"
-		)
-		(instances
-			(project "miniCO2"
-				(path "/4716ccc0-88a0-4c42-87c9-ed1e02729e90/03971f06-80f4-45fd-a837-c09f1f921de9"
-					(reference "D5")
-					(unit 1)
-				)
-			)
-		)
-	)
-	(symbol
 		(lib_name "GND_1")
 		(lib_id "power:GND")
@@
 			)
 		)
-		(property "LCSC Part #" "C274341"
+		(property "LCSC Part #" "C270344"
 			(at 72.39 44.45 0)
 			(effects
